File: hardware/MaMaoHub_Schematic.kicad_sch (KiCad schematic)
At the start: 1 part

Commit message: Update: Added professional 3D render and detailed hardware pinout v2.0
Parts:
- added ?: (no value), symbol TTL_RS485
Connections:
- new net: ?.1 (DI), ?.8 (GPIO14_TX)
Other:
- note added: "['at', '100', '150', '0']"
- note added: "['at', '100', '160', '0']"
Changed lines of the file:
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@@
     (title "MaMaoHub - NMEA 0183 Hub")
     (company "PZero Hubs")
-    (comment 1 "Raspberry Pi Zero 2 W Based")
+    (rev "v2.0")
+    (comment 1 "Final Wiring and Physical Routing")
+    (comment 2 "Includes 3D Layout Components")
   )
-  (symbol (lib_id "RPi_Zero_2W") (at 100 100 0) (unit 1)
-    (in_bom yes) (on_board yes) (fields_autoplaced)
+  (symbol (lib_id "RPi_Zero_2W") (at 50 100 0) (unit 1)
+    (in_bom yes) (on_board yes)
   )
-  (wire (pts (xy 110 100) (xy 130 100))
+  (symbol (lib_id "TTL_RS485") (at 120 100 0) (unit 1)
+    (in_bom yes) (on_board yes)
   )
-  (comment (at 50 200 0) (effects (font (size 2 2))) (text "NOTE: UART TX (GPIO 14) connects to TTL-RS485 DI for Multiplex A+B output."))
+  (wire (pts (xy 55.08 100) (xy 114.92 100))) # RPi TX to TTL DI
+  (text (at 100 150 0) (effects (font (size 2 2))) (text "M3: Navigatore Out (A+ / B-) from TTL Module"))
+  (text (at 100 160 0) (effects (font (size 2 2))) (text "P1-P3: Waveshare USB connections to RPi"))
 )
